Commit message: reconfigured urdfs

File: ros_ws/src/virtual_tactile_pad/urdf/panda_arm.urdf (robot description, URDF)
Before this commit: robot panda, 8 links, 7 joints
Links:
- added link panda_link8, mass 0.0
- link panda_link0: mass 2.8142028896 -> 0.629769
- link panda_link1: mass 2.3599995791 -> 4.970684
- link panda_link2: mass 2.379518833 -> 0.646926
- link panda_link3: mass 2.6498823337 -> 3.228604
- link panda_link4: mass 2.6948018744 -> 3.587895
- link panda_link5: mass 2.9812816864 -> 1.225946
- link panda_link6: mass 1.1285806309 -> 1.666555
- link panda_link7: mass 0.4052912465 -> 7.35522e-01
Joints:
- added joint panda_joint8: type fixed, parent panda_link7, child panda_link8, origin xyz=0 0 0.107 rpy=0 0 0, axis 0 0 0
- joint panda_joint6: limit lower=-0.0175 upper=3.752 effort=12 velocity=2.6100 -> lower=-0.0175 upper=3.7525 effort=12 velocity=2.6100; origin xyz=0 0 0 rpy=-1.57079632679 0 0 -> xyz=0 0 0 rpy=1.57079632679 0 0

Commit message: ordering urdfs

File: ros_ws/src/virtual_tactile_pad/urdf/panda_arm.urdf (robot description, URDF)
Before this commit: robot panda, 9 links, 8 joints
Links:
- added link ati_net_gamma, mass 1.145; collision mesh filename=package://virtual_tactile_pad/urdf/meshes/ati_net_gamma.stl; visual mesh filename=package://virtual_tactile_pad/urdf/meshes/ati_net_gamma.stl
- added link mounting_pad, mass 0.184292; collision mesh filename=package://virtual_tactile_pad/urdf/meshes/mounting_pad.stl; visual mesh filename=package://virtual_tactile_pad/urdf/meshes/mounting_pad.stl
- added link pad, mass 0.145376; collision mesh filename=package://virtual_tactile_pad/urdf/meshes/pad.stl; visual mesh filename=package://virtual_tactile_pad/urdf/meshes/pad.stl
Joints:
- added joint ati_net_gamma_to_mounting_pad: type fixed, parent ati_net_gamma, child mounting_pad, origin xyz=0 0 -0.0146 rpy=0 3.141592654 1.047
- added joint mounting_pad_to_pad: type fixed, parent mounting_pad, child pad, origin xyz=0 0 0 rpy=0 0 0.
- added joint panda_joint_to_ati_gamma: type fixed, parent panda_link8, child ati_net_gamma, origin xyz=0 0 0 rpy=0 3.141592654 1.05398163
- joint panda_joint6: origin xyz=0 0 0 rpy=1.57079632679 0 0 -> xyz=0 0 0 rpy=1.57079632679 3.141592654 0
- joint panda_joint8: origin xyz=0 0 0.107 rpy=0 0 0 -> xyz=0 0 0.107 rpy=0 0 -1.57079632679

Commit message: new stuffs

File: ros_ws/src/virtual_tactile_pad/urdf/panda_arm.urdf (robot description, URDF)
Before this commit: robot panda, 12 links, 11 joints
Joints:
- joint ati_net_gamma_to_mounting_pad: origin xyz=0 0 -0.0146 rpy=0 3.141592654 1.047 -> xyz=0 0 -0.0146 rpy=0 3.141592654 0
- joint panda_joint_to_ati_gamma: origin xyz=0 0 0 rpy=0 3.141592654 0 -> xyz=0 0 0.0287 rpy=0 3.141592654 0

File: ros_ws/src/virtual_tactile_pad/urdf/panda_arm.urdf.xacro (robot description, xacro)
@@ -244,5 +244,5 @@
         <link name="ati_net_gamma">
             <visual>
-                <origin xyz="0 0 0" rpy="0 0 0.5" />
+                <origin xyz="0 0 0" rpy="0 0 0.523796327" />
                 <geometry>
                     <mesh filename="package://virtual_tactile_pad/urdf/meshes/ati_net_gamma.stl" />
@@ -251,5 +251,5 @@
             </visual>
             <collision>
-                <origin xyz="0 0 0" rpy="0 0 0.5" />
+                <origin xyz="0 0 0" rpy="0 0 0.523796327" />
                 <geometry>
                     <mesh filename="package://virtual_tactile_pad/urdf/meshes/ati_net_gamma.stl" />
@@ -258,5 +258,5 @@
             <inertial>
                 <mass value="1.145" />
-                <origin xyz="0 0 0" rpy="0 0 0.5" />
+                <origin xyz="0 0 0" rpy="0 0 0.523796327" />
                 <inertia ixx="0.4644" ixy="0.035" ixz="0.00153" iyy="0.6389" iyz="0.00056" izz="0.9040" />
             </inertial>
@@ -289,5 +289,5 @@
             <parent link="ati_net_gamma" />
             <child link="mounting_pad" />
-            <origin xyz="0 0 -0.0146" rpy="0 3.141592654 -0.023796327" />
+            <origin xyz="0 0 -0.0146" rpy="0 3.141592654 0" />
         </joint>
     </xacro:if>
