Commit message: ordering launch files

File: ros_ws/src/virtual_tactile_pad/urdf/panda_arm.urdf.xacro (robot description, xacro)
@@ -1,4 +1,6 @@
 <?xml version="1.0"?>
 <robot name="panda" xmlns:xacro="http://www.ros.org/wiki/xacro">
+    <!-- Add argument for FT sensor -->
+    <xacro:arg name="use_ft_sensor" default="false"/>
     <!-- panda Links -->
     <link name="panda_link0">
@@ -237,54 +239,84 @@
         <axis xyz="0 0 0" />
     </joint>
-    <!-- ati-net-gamma Link -->
-    <link name="ati_net_gamma">
-        <visual>
-            <origin xyz="0 0 0" rpy="0 0 0" />
-            <geometry>
-                <mesh filename="package://virtual_tactile_pad/urdf/meshes/ati_net_gamma.stl" />
-            </geometry>
-            <material name="ati_net_gamma_gray" />
-        </visual>
-        <collision>
-            <origin xyz="0 0 0" rpy="0 0 0" />
-            <geometry>
-                <mesh filename="package://virtual_tactile_pad/urdf/meshes/ati_net_gamma.stl" />
-            </geometry>
-        </collision>
-        <inertial>
-            <mass value="1.145" />
-            <origin xyz="0 0 0" rpy="0 0 0" />
-            <inertia ixx="0.4644" ixy="0.035" ixz="0.00153" iyy="0.6389" iyz="0.00056" izz="0.9040" />
-        </inertial>
-    </link>
-    <joint name="panda_joint_to_ati_gamma" type="fixed">
-        <parent link="panda_link8" />
-        <child link="ati_net_gamma" />
-        <origin xyz="0 0 0" rpy="0 3.141592654 1.05398163" />
-    </joint>
-    <!-- Mounting Pad Link -->
-    <link name="mounting_pad">
-        <visual>
-            <geometry>
-                <mesh filename="package://virtual_tactile_pad/urdf/meshes/mounting_pad.stl" />
-            </geometry>
-            <material name="mounting_pad_gray" />
-        </visual>
-        <collision>
-            <geometry>
-                <mesh filename="package://virtual_tactile_pad/urdf/meshes/mounting_pad.stl" />
-            </geometry>
-        </collision>
-        <inertial>
-            <mass value="0.184292" />
-            <inertia ixx="0.0000361368" ixy="0.0" ixz="0.0" iyy="0.000046691" iyz="0.0"
-                izz="0.00007688" />
-        </inertial>
-    </link>
-    <joint name="ati_net_gamma_to_mounting_pad" type="fixed">
-        <parent link="ati_net_gamma" />
-        <child link="mounting_pad" />
-        <origin xyz="0 0 -0.0146" rpy="0 3.141592654 1.047" />
-    </joint>
+    <!-- Conditionally include FT sensor or direct mounting -->
+    <xacro:if value="$(arg use_ft_sensor)">
+        <!-- ati-net-gamma Link -->
+        <link name="ati_net_gamma">
+            <visual>
+                <origin xyz="0 0 0" rpy="0 0 0" />
+                <geometry>
+                    <mesh filename="package://virtual_tactile_pad/urdf/meshes/ati_net_gamma.stl" />
+                </geometry>
+                <material name="ati_net_gamma_gray" />
+            </visual>
+            <collision>
+                <origin xyz="0 0 0" rpy="0 0 0" />
+                <geometry>
+                    <mesh filename="package://virtual_tactile_pad/urdf/meshes/ati_net_gamma.stl" />
+                </geometry>
+            </collision>
+            <inertial>
+                <mass value="1.145" />
+                <origin xyz="0 0 0" rpy="0 0 0" />
+                <inertia ixx="0.4644" ixy="0.035" ixz="0.00153" iyy="0.6389" iyz="0.00056" izz="0.9040" />
+            </inertial>
+        </link>
+        <joint name="panda_joint_to_ati_gamma" type="fixed">
+            <parent link="panda_link8" />
+            <child link="ati_net_gamma" />
+            <origin xyz="0 0 0" rpy="0 3.141592654 1.05398163" />
+        </joint>
+        <!-- Mounting Pad Link -->
+        <link name="mounting_pad">
+            <visual>
+                <geometry>
+                    <mesh filename="package://virtual_tactile_pad/urdf/meshes/mounting_pad.stl" />
+                </geometry>
+                <material name="mounting_pad_gray" />
+            </visual>
+            <collision>
+                <geometry>
+                    <mesh filename="package://virtual_tactile_pad/urdf/meshes/mounting_pad.stl" />
+                </geometry>
+            </collision>
+            <inertial>
+                <mass value="0.184292" />
+                <inertia ixx="0.0000361368" ixy="0.0" ixz="0.0" iyy="0.000046691" iyz="0.0"
+                    izz="0.00007688" />
+            </inertial>
+        </link>
+        <joint name="ati_net_gamma_to_mounting_pad" type="fixed">
+            <parent link="ati_net_gamma" />
+            <child link="mounting_pad" />
+            <origin xyz="0 0 -0.0146" rpy="0 3.141592654 1.047" />
+        </joint>
+    </xacro:if>
+    <xacro:unless value="$(arg use_ft_sensor)">
+        <!-- Mounting Pad Link -->
+        <link name="mounting_pad">
+            <visual>
+                <geometry>
+                    <mesh filename="package://virtual_tactile_pad/urdf/meshes/mounting_pad.stl" />
+                </geometry>
+                <material name="mounting_pad_gray" />
+            </visual>
+            <collision>
+                <geometry>
+                    <mesh filename="package://virtual_tactile_pad/urdf/meshes/mounting_pad.stl" />
+                </geometry>
+            </collision>
+            <inertial>
+                <mass value="0.184292" />
+                <inertia ixx="0.0000361368" ixy="0.0" ixz="0.0" iyy="0.000046691" iyz="0.0"
+                    izz="0.00007688" />
+            </inertial>
+        </link>
+        <!-- Direct joint from panda_link8 to mounting_pad -->
+        <joint name="panda_link8_to_mounting_pad" type="fixed">
+            <parent link="panda_link8" />
+            <child link="mounting_pad" />
+            <origin xyz="0 0 0" rpy="0 0 0" />  <!-- Adjusted rpy to account for no sensor -->
+        </joint>
+    </xacro:unless>
     <!-- Pad Link -->
     <link name="pad">

Commit message: important modif

File: ros_ws/src/virtual_tactile_pad/urdf/panda_arm.urdf.xacro (robot description, xacro)
@@ -244,5 +244,5 @@
         <link name="ati_net_gamma">
             <visual>
-                <origin xyz="0 0 0" rpy="0 0 0" />
+                <origin xyz="0 0 0" rpy="0 0 0.5" />
                 <geometry>
                     <mesh filename="package://virtual_tactile_pad/urdf/meshes/ati_net_gamma.stl" />
@@ -251,5 +251,5 @@
             </visual>
             <collision>
-                <origin xyz="0 0 0" rpy="0 0 0" />
+                <origin xyz="0 0 0" rpy="0 0 0.5" />
                 <geometry>
                     <mesh filename="package://virtual_tactile_pad/urdf/meshes/ati_net_gamma.stl" />
@@ -258,5 +258,5 @@
             <inertial>
                 <mass value="1.145" />
-                <origin xyz="0 0 0" rpy="0 0 0" />
+                <origin xyz="0 0 0" rpy="0 0 0.5" />
                 <inertia ixx="0.4644" ixy="0.035" ixz="0.00153" iyy="0.6389" iyz="0.00056" izz="0.9040" />
             </inertial>
@@ -265,5 +265,5 @@
             <parent link="panda_link8" />
             <child link="ati_net_gamma" />
-            <origin xyz="0 0 0" rpy="0 3.141592654 1.05398163" />
+            <origin xyz="0 0 0.0187" rpy="0 3.141592654 0.0" />
         </joint>
         <!-- Mounting Pad Link -->
@@ -289,5 +289,5 @@
             <parent link="ati_net_gamma" />
             <child link="mounting_pad" />
-            <origin xyz="0 0 -0.0146" rpy="0 3.141592654 1.047" />
+            <origin xyz="0 0 -0.0146" rpy="0 3.141592654 -0.023796327" />
         </joint>
     </xacro:if>
@@ -316,5 +316,5 @@
             <parent link="panda_link8" />
             <child link="mounting_pad" />
-            <origin xyz="0 0 0" rpy="0 0 0" />  <!-- Adjusted rpy to account for no sensor -->
+            <origin xyz="0 0 0" rpy="0 0 0" />
         </joint>
     </xacro:unless>

Commit message: update launch files to launch with franka-ros

File: ros_ws/src/virtual_tactile_pad/urdf/panda_arm.urdf.xacro (robot description, xacro)
@@ -190,5 +190,5 @@
         <safety_controller k_position="100.0" k_velocity="40.0" soft_lower_limit="-0.0175"
             soft_upper_limit="3.7525" />
-        <origin rpy="1.57079632679 3.141592654 0" xyz="0 0 0" />
+        <origin rpy="1.57079632679 0 0" xyz="0 0 0" />
         <parent link="panda_link5" />
         <child link="panda_link6" />

Commit message: added good panda localization

File: ros_ws/src/virtual_tactile_pad/urdf/panda_arm.urdf.xacro (robot description, xacro)
@@ -265,5 +265,5 @@
             <parent link="panda_link8" />
             <child link="ati_net_gamma" />
-            <origin xyz="0 0 0.0187" rpy="0 3.141592654 0.0" />
+            <origin xyz="0 0 0.0287" rpy="0 3.141592654 0" />
         </joint>
         <!-- Mounting Pad Link -->

Commit message: added adapter

File: ros_ws/src/virtual_tactile_pad/urdf/panda_arm.urdf.xacro (robot description, xacro)
@@ -2,5 +2,5 @@
 <robot name="panda" xmlns:xacro="http://www.ros.org/wiki/xacro">
     <!-- Add argument for FT sensor -->
-    <xacro:arg name="use_ft_sensor" default="false"/>
+    <xacro:arg name="use_ft_sensor" default="false" />
     <!-- panda Links -->
     <link name="panda_link0">
@@ -241,4 +241,31 @@
     <!-- Conditionally include FT sensor or direct mounting -->
     <xacro:if value="$(arg use_ft_sensor)">
+        <!-- adapter link -->
+        <link name="adapter">
+            <visual>
+                <origin xyz="0 0 0" rpy="0 0 0" />
+                <geometry>
+                    <mesh filename="package://virtual_tactile_pad/urdf/meshes/adapter.stl" />
+                </geometry>
+                <material name="adapter_gray" />
+            </visual>
+            <collision>
+                <origin xyz="0 0 0" rpy="0 0 0" />
+                <geometry>
+                    <mesh filename="package://virtual_tactile_pad/urdf/meshes/adapter.stl" />
+                </geometry>
+            </collision>
+            <inertial>
+                <mass value="0.157201" />
+                <origin xyz="0 0 0" rpy="0 0 0" />
+                <inertia ixx="7.5980706e-5" ixy="0" ixz="6.2031582e-5" iyy="0" iyz="0"
+                    izz="1.309e-4" />
+            </inertial>
+        </link>
+        <joint name="panda_joint_to_adapter" type="fixed">
+            <parent link="panda_link8" />
+            <child link="adapter" />
+            <origin xyz="0 0 0" rpy="0 0 0" />
+        </joint>
         <!-- ati-net-gamma Link -->
         <link name="ati_net_gamma">
@@ -259,11 +286,12 @@
                 <mass value="1.145" />
                 <origin xyz="0 0 0" rpy="0 0 0.523796327" />
-                <inertia ixx="0.4644" ixy="0.035" ixz="0.00153" iyy="0.6389" iyz="0.00056" izz="0.9040" />
+                <inertia ixx="0.4644" ixy="0.035" ixz="0.00153" iyy="0.6389" iyz="0.00056"
+                    izz="0.9040" />
             </inertial>
         </link>
         <joint name="panda_joint_to_ati_gamma" type="fixed">
-            <parent link="panda_link8" />
+            <parent link="adapter" />
             <child link="ati_net_gamma" />
-            <origin xyz="0 0 0.0287" rpy="0 3.141592654 0" />
+            <origin xyz="0 0 0.034" rpy="0 3.141592654 0" />
         </joint>
         <!-- Mounting Pad Link -->
@@ -281,7 +309,7 @@
             </collision>
             <inertial>
-                <mass value="0.184292" />
-                <inertia ixx="0.0000361368" ixy="0.0" ixz="0.0" iyy="0.000046691" iyz="0.0"
-                    izz="0.00007688" />
+                <mass value="0.064186" />
+                <inertia ixx="1.2643e-5" ixy="0.0" ixz="0.0" iyy="1.6296014e-5" iyz="0.0"
+                    izz="2.6868247e-5" />
             </inertial>
         </link>
@@ -307,7 +335,7 @@
             </collision>
             <inertial>
-                <mass value="0.184292" />
-                <inertia ixx="0.0000361368" ixy="0.0" ixz="0.0" iyy="0.000046691" iyz="0.0"
-                    izz="0.00007688" />
+                <mass value="0.064186" />
+                <inertia ixx="1.2643e-5" ixy="0.0" ixz="0.0" iyy="1.6296014e-5" iyz="0.0"
+                    izz="2.6868247e-5" />
             </inertial>
         </link>
@@ -334,5 +362,5 @@
         <inertial>
             <mass value="0.145376" />
-            <inertia ixx="0.0002345" ixy="0.0" ixz="0.0" iyy="0.0004074" iyz="0.0" izz="0.0001733" />
+            <inertia ixx="2.345e-4" ixy="0.0" ixz="0.0" iyy="4.074e-4" iyz="0.0" izz="1.733e-4" />
         </inertial>
     </link>
@@ -358,3 +386,6 @@
         <color rgba="0.4 0.4 0.4 1." />
     </material>
+    <material name="adapter_gray">
+        <color rgba="0.5 0.5 0.5 1." />
+    </material>
 </robot>

Commit message: modify ati inertia

File: ros_ws/src/virtual_tactile_pad/urdf/panda_arm.urdf.xacro (robot description, xacro)
@@ -284,8 +284,8 @@
             </collision>
             <inertial>
-                <mass value="1.145" />
+                <mass value="0.335594" />
                 <origin xyz="0 0 0" rpy="0 0 0.523796327" />
-                <inertia ixx="0.4644" ixy="0.035" ixz="0.00153" iyy="0.6389" iyz="0.00056"
-                    izz="0.9040" />
+                <inertia ixx="1.479e-4" ixy="0" ixz="0" iyy="2.071e-4" iyz="0"
+                    izz="2.918e-4" />
             </inertial>
         </link>

Commit message: modify xacro

File: ros_ws/src/virtual_tactile_pad/urdf/panda_arm.urdf.xacro (robot description, xacro)
@@ -293,5 +293,5 @@
             <parent link="adapter" />
             <child link="ati_net_gamma" />
-            <origin xyz="0 0 0.034" rpy="0 3.141592654 0" />
+            <origin xyz="0 0 0.0287" rpy="0 3.141592654 0" />
         </joint>
         <!-- Mounting Pad Link -->

Commit message: added controller

File: ros_ws/src/virtual_tactile_pad/urdf/panda_arm.urdf.xacro (robot description, xacro)
@@ -250,10 +250,4 @@
                 <material name="adapter_gray" />
             </visual>
-            <collision>
-                <origin xyz="0 0 0" rpy="0 0 0" />
-                <geometry>
-                    <mesh filename="package://virtual_tactile_pad/urdf/meshes/adapter.stl" />
-                </geometry>
-            </collision>
             <inertial>
                 <mass value="0.157201" />
@@ -277,10 +271,4 @@
                 <material name="ati_net_gamma_gray" />
             </visual>
-            <collision>
-                <origin xyz="0 0 0" rpy="0 0 0.523796327" />
-                <geometry>
-                    <mesh filename="package://virtual_tactile_pad/urdf/meshes/ati_net_gamma.stl" />
-                </geometry>
-            </collision>
             <inertial>
                 <mass value="0.335594" />
@@ -303,9 +291,4 @@
                 <material name="mounting_pad_gray" />
             </visual>
-            <collision>
-                <geometry>
-                    <mesh filename="package://virtual_tactile_pad/urdf/meshes/mounting_pad.stl" />
-                </geometry>
-            </collision>
             <inertial>
                 <mass value="0.064186" />
@@ -329,9 +312,4 @@
                 <material name="mounting_pad_gray" />
             </visual>
-            <collision>
-                <geometry>
-                    <mesh filename="package://virtual_tactile_pad/urdf/meshes/mounting_pad.stl" />
-                </geometry>
-            </collision>
             <inertial>
                 <mass value="0.064186" />
@@ -355,9 +333,4 @@
             <material name="pad_blue" />
         </visual>
-        <collision>
-            <geometry>
-                <mesh filename="package://virtual_tactile_pad/urdf/meshes/pad.stl" />
-            </geometry>
-        </collision>
         <inertial>
             <mass value="0.145376" />
